File: pmodThingy.kicad_pcb (KiCad board)
At the start: 2 copper layers, 58.3 x 47.1 mm, 23 parts, among them J1 PMOD_A, J2 PMOD_B, J3 USB_B_Micro, J4 PMOD_passthrough, J5 ICSP, J6 Conn_Coaxial_Power, U1 ATmega32U4-A, U2 AMS1117-3.3, Y1 8MHz

Commit message: relabel some pins on schematic
Connections:
- net /IO1 renamed /IO1_SCK
- net /IO2_SS renamed /IO2_MOSI
- net /IO3_MOSI renamed /IO3_MISO
- net /IO4_MISO renamed /IO4
- net /IO5_SCK renamed /IO5
- J6 pad S2: GND -> (no net)
- J6 pad S3: GND -> (no net)
- J6 pad S4: GND -> (no net)
