File: pmodThingy.kicad_sch (KiCad schematic)
At the start: 23 parts, among them J1 PMOD_A, J2 PMOD_B, J3 USB_B_Micro, J4 PMOD_passthrough, J5 ICSP, J6 Conn_Coaxial_Power, U1 ATmega32U4-A, U2 AMS1117-3.3, Y1 8MHz

Commit message: relabel some pins on schematic
Connections:
- net IO1 renamed IO1_SCK
- net IO2_SS renamed IO2_MOSI
- net IO3_MOSI renamed IO3_MISO
- net IO4_MISO renamed IO4
- net IO5_SCK renamed IO5
Changed lines of the file:
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@@
     (effects (font (size 1.27 1.27)) (justify left bottom))
   )
-  (label "IO1" (at 241.3 59.055 0) (fields_autoplaced)
+  (label "IO1_SCK" (at 241.3 59.055 0) (fields_autoplaced)
     (effects (font (size 1.27 1.27)) (justify left bottom))
   )
-  (label "IO1" (at 34.925 92.075 0) (fields_autoplaced)
+  (label "IO1_SCK" (at 34.925 92.075 0) (fields_autoplaced)
     (effects (font (size 1.27 1.27)) (justify left bottom))
   )
@@
     (effects (font (size 1.27 1.27)) (justify left bottom))
   )
-  (label "IO3_MOSI" (at 241.3 64.135 0) (fields_autoplaced)
+  (label "IO3_MISO" (at 241.3 64.135 0) (fields_autoplaced)
     (effects (font (size 1.27 1.27)) (justify left bottom))
   )
@@
     (effects (font (size 1.27 1.27)) (justify left bottom))
   )
-  (label "IO4_MISO" (at 34.925 99.695 0) (fields_autoplaced)
+  (label "IO4" (at 34.925 99.695 0) (fields_autoplaced)
     (effects (font (size 1.27 1.27)) (justify left bottom))
   )
@@
     (effects (font (size 1.27 1.27)) (justify left bottom))
   )
-  (label "IO3_MOSI" (at 34.925 97.155 0) (fields_autoplaced)
+  (label "IO3_MISO" (at 34.925 97.155 0) (fields_autoplaced)
     (effects (font (size 1.27 1.27)) (justify left bottom))
   )
-  (label "IO2_SS" (at 241.3 61.595 0) (fields_autoplaced)
+  (label "IO2_MOSI" (at 241.3 61.595 0) (fields_autoplaced)
     (effects (font (size 1.27 1.27)) (justify left bottom))
   )
-  (label "IO5_SCK" (at 56.515 27.94 0) (fields_autoplaced)
+  (label "IO5" (at 56.515 27.94 0) (fields_autoplaced)
     (effects (font (size 1.27 1.27)) (justify left bottom))
   )
@@
     (effects (font (size 1.27 1.27)) (justify left bottom))
   )
-  (label "IO5_SCK" (at 241.3 69.215 0) (fields_autoplaced)
+  (label "IO5" (at 241.3 69.215 0) (fields_autoplaced)
     (effects (font (size 1.27 1.27)) (justify left bottom))
   )
@@
     (effects (font (size 1.27 1.27)) (justify left bottom))
   )
-  (label "IO4_MISO" (at 85.09 120.015 180) (fields_autoplaced)
+  (label "IO4" (at 85.09 120.015 180) (fields_autoplaced)
     (effects (font (size 1.27 1.27)) (justify right bottom))
   )
@@
     (effects (font (size 1.27 1.27)) (justify left bottom))
   )
-  (label "IO2_SS" (at 34.925 94.615 0) (fields_autoplaced)
+  (label "IO2_MOSI" (at 34.925 94.615 0) (fields_autoplaced)
     (effects (font (size 1.27 1.27)) (justify left bottom))
   )
-  (label "IO5_SCK" (at 85.09 122.555 180) (fields_autoplaced)
+  (label "IO5" (at 85.09 122.555 180) (fields_autoplaced)
     (effects (font (size 1.27 1.27)) (justify right bottom))
   )
@@
     (effects (font (size 1.27 1.27)) (justify left bottom))
   )
-  (label "IO4_MISO" (at 241.3 66.675 0) (fields_autoplaced)
+  (label "IO4" (at 241.3 66.675 0) (fields_autoplaced)
     (effects (font (size 1.27 1.27)) (justify left bottom))
   )
@@
     (effects (font (size 1.27 1.27)) (justify left bottom))
   )
-  (label "IO5_SCK" (at 34.925 102.235 0) (fields_autoplaced)
+  (label "IO5" (at 34.925 102.235 0) (fields_autoplaced)
     (effects (font (size 1.27 1.27)) (justify left bottom))
   )
@@
     (effects (font (size 1.27 1.27)) (justify left bottom))
   )
-  (label "IO4_MISO" (at 56.515 25.4 0) (fields_autoplaced)
+  (label "IO4" (at 56.515 25.4 0) (fields_autoplaced)
     (effects (font (size 1.27 1.27)) (justify left bottom))
   )
-  (label "IO3_MOSI" (at 34.925 33.02 180) (fields_autoplaced)
+  (label "IO3_MISO" (at 34.925 33.02 180) (fields_autoplaced)
     (effects (font (size 1.27 1.27)) (justify right bottom))
   )
-  (label "IO1" (at 34.925 27.94 180) (fields_autoplaced)
+  (label "IO1_SCK" (at 34.925 27.94 180) (fields_autoplaced)
     (effects (font (size 1.27 1.27)) (justify right bottom))
   )
@@
     (effects (font (size 1.27 1.27)) (justify left bottom))
   )
-  (label "IO2_SS" (at 34.925 30.48 180) (fields_autoplaced)
+  (label "IO2_MOSI" (at 34.925 30.48 180) (fields_autoplaced)
     (effects (font (size 1.27 1.27)) (justify right bottom))
   )
@@
     (effects (font (size 1.27 1.27)) (justify right bottom))
   )
-  (label "IO3_MOSI" (at 101.6 122.555 0) (fields_autoplaced)
+  (label "IO3_MISO" (at 101.6 122.555 0) (fields_autoplaced)
     (effects (font (size 1.27 1.27)) (justify left bottom))
   )
